File: v2.0/A2DVI.v2.0.kicad_sch (KiCad schematic)
At the start: 31 parts, among them CON3 Apple2_edge_connector, U1 RPI-Pico, U2 74LVC245, U3 74LVC245, U4 74LVC245, U5 74LVC245

Commit message: Add files via upload
Parts:
- D1: value 1N5819 -> MBR120VLSFT1G
Changed lines of the file:
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@@
       (effects (font (size 1.27 1.27)))
     )
-    (property "Value" "1N5819" (at 156.21 19.05 0)
+    (property "Value" "MBR120VLSFT1G" (at 156.21 19.05 0)
       (effects (font (size 1.27 1.27)))
     )
