File: v2.3/A2DVI.v2.3.kicad_pcb (KiCad board)
At the start: 2 copper layers, 111.6 x 57 mm, 78 parts, among them U1 Pico, U2 74HC245, U3 74HC245, U4 74HC245, U5 74HC245

Commit message: Add files via upload
Parts:
- removed C10, C11, C12, C13, C14, C7, C8, C9: 100pF, Capacitor_THT:C_Disc_D3.0mm_W1.6mm_P2.50mm
- added R10: 270, Resistor_THT:R_Axial_DIN0204_L3.6mm_D1.6mm_P5.08mm_Horizontal, F.Cu at (128.2, 110.7)
- added R11: 270, Resistor_THT:R_Axial_DIN0204_L3.6mm_D1.6mm_P5.08mm_Horizontal, F.Cu at (128.2, 113.1)
- added R12: 270, Resistor_THT:R_Axial_DIN0204_L3.6mm_D1.6mm_P5.08mm_Horizontal, F.Cu at (128.2, 115.2)
- added R5: 270, Resistor_THT:R_Axial_DIN0204_L3.6mm_D1.6mm_P5.08mm_Horizontal, F.Cu at (128.2, 99.4)
- added R6: 270, Resistor_THT:R_Axial_DIN0204_L3.6mm_D1.6mm_P5.08mm_Horizontal, F.Cu at (128.2, 101.5)
- added R7: 270, Resistor_THT:R_Axial_DIN0204_L3.6mm_D1.6mm_P5.08mm_Horizontal, F.Cu at (128.2, 104.0)
- added R8: 270, Resistor_THT:R_Axial_DIN0204_L3.6mm_D1.6mm_P5.08mm_Horizontal, F.Cu at (128.2, 106.2)
- added R9: 270, Resistor_THT:R_Axial_DIN0204_L3.6mm_D1.6mm_P5.08mm_Horizontal, F.Cu at (128.2, 108.6)
Routing:
- net CK_N: track 22.0 -> 19.4 mm
- net D1_N: track 30.0 -> 27.4 mm
- net D0_P: track 33.8 -> 31.2 mm
- net D0_N: track 34.5 -> 31.9 mm
- net CK_P: track 23.0 -> 20.4 mm
- net D1_P: track 29.3 -> 26.7 mm
- net D2_N: track 18.6 -> 16.3 mm
- net D2_P: track 17.8 -> 15.6 mm
