File: v2.3/A2DVI.v2.3.kicad_sch (KiCad schematic)
At the start: 28 parts, among them CON3 Apple2_edge_connector, U1 RPI-Pico, U2 74HC245, U3 74HC245, U4 74HC245, U5 74HC245

Commit message: Add files via upload
Parts:
- removed C10, C11, C12, C13, C14, C7, C8, C9: 100p, symbol Device:C
- added R10, R11, R12, R5, R6, R7, R8, R9: 270, Resistor_SMD:R_0402_1005Metric_Pad0.72x0.64mm_HandSolder, symbol Device:R
Connections:
- net CK+: now also R11.2
- net CK-: now also R12.2
- net D0+: now also R9.2
- net D0-: now also R10.2
- net D1+: now also R7.2
- net D2+: now also R5.2
- net D2-: now also R6.2
- net at U1.19 (GP14): now also R11.1
- net at U1.20 (GP15): now also R12.1
- net at U1.21 (GP16): now also R5.1
- net at U1.22 (GP17): now also R6.1
- net at U1.24 (GP18): now also R7.1
- net at U1.25 (GP19): now also R8.1
- net at U1.26 (GP20): now also R9.1
- net at U1.27 (GP21): now also R10.1
- net at DVI1.6: now also R8.2
