File: v4.4/A2DVI.v4.4.kicad_pcb (KiCad board)
At the start: 2 copper layers, 88.6 x 47.2 mm, 131 parts, among them Q1 2N7002, SW1 YTS-A016-X, U1 QFN-56-1EP_7x7mm_P0.4mm_EP3.2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, U2 W25Q16JVUXIQ, U3 SY8089AAAC, SOT-23-5, U4 SN74LVC245APWR, U5 SN74LVC245APWR, U6 SN74LVC245APWR, U7 74LVC1G08, SOT-23-5, U8 74LVC3G34, VSSOP-8_3.0x3.0mm_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

Commit message: Add files via upload
Parts:
- added R28: 5.1k 1%, Resistor_SMD:R_0402_1005Metric, F.Cu at (104.9, 124.5)
- added R29: 100k, Resistor_SMD:R_0402_1005Metric, F.Cu at (101.0, 121.0)
- moved R10 1.26 mm to (101.7, 124.5)
- moved R9 1.10 mm to (101.7, 125.5)
- moved R11 0.87 mm to (104.9, 125.5)
Connections:
- R10 pad 1: FB -> FB1
Routing:
- net SW: track 9.90 -> 13.1 mm
- net FB1: track 0.00 -> 2.17 mm
- net 3.3V: track 291.7 -> 289.7 mm
- net GND: track 160.3 -> 158.7 mm, vias 166 -> 163
- net VSYS: track 22.9 -> 21.8 mm
- net 3.3V-en: track 2.73 -> 1.79 mm
Other:
- board text added: ""
- board text removed: "<-KBD"
- board text removed: "KBD->"
