File: v4.4/A2DVI.v4.4.kicad_sch (KiCad schematic)
At the start: 68 parts, among them CON3 Apple2_edge_connector, Q1 2N7002, SW1 SW_Push, U3 SY8089AAAC, U4 74LVC245, U5 74LVC245, U6 74LVC245, U7 74LVC1G08, U7 W25Q16JVSS, U8 74LVC3G34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

Commit message: Add files via upload
Parts:
- added R28: 4.7k, Resistor_SMD:R_0402_1005Metric_Pad0.72x0.64mm_HandSolder, symbol Device:R
- added R29: 50k, Resistor_SMD:R_0402_1005Metric_Pad0.72x0.64mm_HandSolder, symbol Device:R
- R11: value 50k -> 49.9k
Connections:
- net +3V3: now also R29.2
- net at R11.1, U3.5 (FB): now also R28.1; no longer R10.1
- net at R3.1, SW1.2: now also R29.1
- new net: R10.1, R28.2
Other:
- moved on the sheet: C13, R10, R11, R9, U3
