File: v5.x/A2DVI.v5.1.kicad_sch (KiCad schematic)
At the start: 19 parts, among them J1 AppleIIBus, U1 CPB

Commit message: Add files via upload
Connections:
- net CK+ is gone; now on net CLK+: R7.1
- net CK- is gone; now on net CLK-: R8.1
- net RUN: no longer names the net of R9.1, U1.30 (Pin_30)
Other:
- moved on the sheet: C2, FU1, H1, H2, H3, R1, R2, R3, R4, R5, R6, R7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
