File: v5.x/A2DVI.v5.1.kicad_pcb (KiCad board)
At the start: 4 copper layers, 65.5 x 79.8 mm, 69 parts, among them U1 CPB

Commit message: Add files via upload
Parts:
- moved C1 0.81 mm to (123.9, 100.4)
- moved R9 0.81 mm to (128.1, 100.4)
- moved D1 0.81 mm to (119.2, 100.4)
Routing:
- net VSYS: track 13.8 -> 15.0 mm
- net ~{IOStr}: track 25.6 -> 25.1 mm
- net GND: track 25.9 -> 25.8 mm, vias 119 -> 118
Changed lines of the file:
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@@
 	(footprint "Diode_SMD:D_SOD-123F"
 		(layer "F.Cu")
-		(at 119.1768 101.1682)
+		(at 119.1768 100.3554)
 		(descr "D_SOD-123F")
 		(tags "D_SOD-123F")
@@
 	(footprint "Resistor_SMD:R_0402_1005Metric"
 		(layer "F.Cu")
-		(at 128.0922 101.1936 180)
+		(at 128.0922 100.3808 180)
 		(descr "Resistor SMD 0402 (1005 Metric), square (rectangular) end terminal, IPC_7351 nominal, (Body size source: IPC-SM-782 page 72, https://www.pcb-3d.com/wordpress/wp-content/uploads/ipc-sm-782a_amendment_1_and_2.pdf), generated with kicad-footprint-generator")
 		(tags "resistor")
@@
 	(footprint "Capacitor_SMD:C_0402_1005Metric_Pad0.74x0.62mm_HandSolder"
 		(layer "F.Cu")
-		(at 123.8504 101.1936 180)
+		(at 123.8504 100.3808 180)
 		(descr "Capacitor SMD 0402 (1005 Metric), square (rectangular) end terminal, IPC_7351 nominal with elongated pad for handsoldering. (Body size source: IPC-SM-782 page 76, https://www.pcb-3d.com/wordpress/wp-content/uploads/ipc-sm-782a_amendment_1_and_2.pdf), generated with kicad-footprint-generator")
 		(tags "capacitor handsolder")
@@
 		)
 	)
+	(gr_rect
+		(start 154.2126 85.2078)
+		(end 165.0746 98.0278)
+		(stroke
+			(width 0.2)
+			(type solid)
+		)
+		(fill solid)
+		(layer "F.SilkS")
+	)
 	(gr_line
 		(start 177.546 138.557)
@@
 	)
 	(via
-		(at 151.1046 131.3688)
-		(size 0.8)
-		(drill 0.4)
-		(layers "F.Cu" "B.Cu")
-		(free yes)
-		(net 1)
-	)
-	(via
 		(at 152.2222 61.5188)
 		(size 0.8)
@@
 	)
 	(segment
-		(start 168.91 116.332)
-		(end 168.8338 116.332)
-		(width 0.2)
-		(layer "B.Cu")
-		(net 1)
-	)
-	(segment
-		(start 123.8504 103.777)
-		(end 123.8504 105.537)
+		(start 127.5822 100.3808)
+		(end 127.2466 100.3808)
 		(width 0.4)
 		(layer "F.Cu")
@@
 	)
 	(segment
-		(start 126.4338 101.1936)
+		(start 127.2466 100.3808)
 		(end 123.8504 103.777)
 		(width 0.4)
@@
 	)
 	(segment
-		(start 127.5822 101.1936)
-		(end 126.4338 101.1936)
+		(start 123.8504 103.777)
+		(end 123.8504 105.537)
 		(width 0.4)
 		(layer "F.Cu")
@@
 	)
 	(segment
-		(start 116.28105 105.48635)
-		(end 116.2304 105.537)
+		(start 117.7768 100.3554)
+		(end 117.7768 101.032896)
 		(width 0.6)
 		(layer "F.Cu")
@@
 	)
 	(segment
-		(start 117.7768 101.1682)
-		(end 116.28105 102.66395)
-		(width 0.6)
+		(start 118.0084 100.3554)
+		(end 121.3104 103.6574)
+		(width 0.2)
 		(layer "F.Cu")
 		(net 3)
 	)
 	(segment
-		(start 121.3104 103.6574)
-		(end 118.8212 101.1682)
+		(start 117.7768 100.3554)
+		(end 118.0084 100.3554)
 		(width 0.2)
 		(layer "F.Cu")
@@
 	)
 	(segment
-		(start 118.8212 101.1682)
-		(end 117.7768 101.1682)
-		(width 0.2)
+		(start 116.28105 102.528646)
+		(end 116.28105 105.48635)
+		(width 0.6)
 		(layer "F.Cu")
 		(net 3)
 	)
 	(segment
-		(start 116.2304 103.177)
+		(start 116.28105 105.48635)
 		(end 116.2304 105.537)
 		(width 0.6)
@@
 	)
 	(segment
-		(start 116.28105 102.66395)
-		(end 116.28105 105.48635)
+		(start 116.2304 103.177)
+		(end 116.2304 105.537)
 		(width 0.6)
 		(layer "F.Cu")
@@
 	)
 	(segment
-		(start 121.3104 105.537)
-		(end 121.3104 103.6574)
+		(start 121.3104 103.6574)
+		(end 121.3104 105.537)
 		(width 0.2)
 		(layer "F.Cu")
@@
 	)
 	(segment
-		(start 123.2829 101.1936)
-		(end 121.56155 101.1936)
+		(start 117.7768 101.032896)
+		(end 116.28105 102.528646)
+		(width 0.6)
+		(layer "F.Cu")
+		(net 3)
+	)
+	(segment
+		(start 123.339475 100.3808)
+		(end 121.618125 100.3808)
 		(width 0.6)
 		(layer "F.Cu")
@@
 	)
 	(segment
-		(start 121.56155 101.1936)
-		(end 121.53615 101.1682)
-		(width 0.6)
-		(layer "F.Cu")
-		(net 4)
-	)
-	(segment
-		(start 121.53615 101.1682)
-		(end 120.5768 101.1682)
+		(start 121.592725 100.3554)
+		(end 120.633375 100.3554)
 		(width 0.6)
 		(layer "F.Cu")
@@
 	)
 	(via
-		(at 122.301 101.1682)
+		(at 122.301 100.3554)
 		(size 0.8)
 		(drill 0.4)
@@
 	)
 	(via
-		(at 121.53615 101.1682)
+		(at 121.53615 100.3554)
 		(size 0.8)
 		(drill 0.4)
@@
 	)
 	(segment
-		(start 124.6632 103.5304)
-		(end 122.301 101.1682)
-		(width 0.6)
-		(layer "B.Cu")
-		(net 4)
-	)
-	(segment
-		(start 121.56155 101.1936)
-		(end 122.2756 101.1936)
+		(start 125.476 103.5304)
+		(end 176.8856 103.5304)
 		(width 0.6)
 		(layer "B.Cu")
@@
 	(segment
 		(start 176.8856 103.5304)
-		(end 124.6632 103.5304)
-		(width 0.6)
-		(layer "B.Cu")
-		(net 4)
-	)
-	(segment
-		(start 176.8856 103.5304)
 		(end 176.8856 104.648)
 		(width 0.8)
@@
 	)
 	(segment
-		(start 122.2756 101.1936)
-		(end 122.301 101.1682)
+		(start 121.53615 100.3554)
+		(end 122.301 100.3554)
 		(width 0.6)
 		(layer "B.Cu")
@@
 	)
 	(segment
-		(start 121.53615 101.1682)
-		(end 121.56155 101.1936)
+		(start 122.301 100.3554)
+		(end 125.476 103.5304)
 		(width 0.6)
 		(layer "B.Cu")
@@
 	)
 	(segment
-		(start 128.6022 101.1936)
-		(end 136.5504 101.1936)
+		(start 136.5504 101.1936)
+		(end 139.0904 103.7336)
 		(width 0.2)
 		(layer "F.Cu")
@@
 	)
 	(segment
-		(start 136.5504 101.1936)
-		(end 139.0904 103.7336)
+		(start 128.6022 100.3808)
+		(end 129.415 101.1936)
 		(width 0.2)
 		(layer "F.Cu")
@@
 	)
 	(segment
+		(start 129.415 101.1936)
+		(end 136.5504 101.1936)
+		(width 0.2)
+		(layer "F.Cu")
+		(net 32)
+	)
+	(segment
 		(start 164.443791 81.552092)
 		(end 164.801267 81.552092)
@@
 	)
 	(segment
-		(start 149.3774 131.0386)
-		(end 146.7104 128.3716)
+		(start 161.671 131.6482)
+		(end 161.0614 131.0386)
 		(width 0.2)
 		(layer "B.Cu")
@@
 	)
 	(segment
-		(start 161.671 131.6482)
-		(end 161.0614 131.0386)
+		(start 150.3172 131.0386)
+		(end 146.7104 127.4318)
 		(width 0.2)
 		(layer "B.Cu")
@@
 	)
 	(segment
-		(start 161.0614 131.0386)
-		(end 149.3774 131.0386)
+		(start 146.7104 127.4318)
+		(end 146.7104 123.317)
 		(width 0.2)
 		(layer "B.Cu")
@@
 	)
 	(segment
-		(start 146.7104 128.3716)
-		(end 146.7104 123.317)
+		(start 161.0614 131.0386)
+		(end 150.3172 131.0386)
 		(width 0.2)
 		(layer "B.Cu")
@@
 		(hatch edge 0.5)
 		(connect_pads
-			(clearance 0.2)
+			(clearance 0.25)
 		)
 		(min_thickness 0.25)
